Commit message: got a working ros2 control config for victor with fake hardware
tested with:
ros2 launch victor_bringup victor.launch.py use_fake_hardware:=true

File: victor_description/ros2_control/iiwa.r2c_hardware.xacro (robot description, xacro)
@@ -1,149 +1,127 @@
 <?xml version="1.0"?>
 <robot xmlns:xacro="http://www.ros.org/wiki/xacro">
-    <xacro:macro name="victor_r2c_hardware" params="name prefix command_interface robot_ip robot_port initial_positions_file use_sim:=^|false use_fake_hardware:=^|true">
-        <xacro:property name="initial_positions" value="${xacro.load_yaml(initial_positions_file)['initial_positions']}"/>
-        <ros2_control name="${name}" type="system">
-            <xacro:if value="$(arg use_sim)">
-                <hardware>
-                    <plugin>gazebo_ros2_control/GazeboSystem</plugin>
-                </hardware>
+    <xacro:macro name="iiwa_r2c_hardware"
+        params="prefix command_interface">
+        <joint name="${prefix}joint_a1">
+            <command_interface name="${command_interface}" />
+            <xacro:if value="${command_interface == 'position'}">
+                <param name="min">-2.96</param>
+                <param name="max">2.96</param>
             </xacro:if>
-            <xacro:unless value="$(arg use_sim)">
-                <hardware>
-                <xacro:if value="${use_fake_hardware}">
-                    <plugin>fake_components/GenericSystem</plugin>
-                        <param name="state_following_offset">0.0</param>
-                </xacro:if>
-                <xacro:unless value="${use_fake_hardware}">
-                    <plugin>victor_hardware/IiwaFRIHardwareInterface</plugin>
-                    <param name="robot_ip">${robot_ip}</param>
-                    <param name="robot_port">${robot_port}</param>
-                    <param name="velocity_filter_cutoff_freq">40</param>
-                    <param name="torque_filter_cutoff_freq">40</param>
-                </xacro:unless>
-                </hardware>
-            </xacro:unless>
-            <joint name="${prefix}joint_a1">
-                <command_interface name="${command_interface}" />
-                    <xacro:if value="${command_interface == 'position'}">
-                        <param name="min">-2.96</param>
-                        <param name="max">2.96</param>
-                    </xacro:if>
-                <state_interface name="position">
-                    <param name="initial_value">${initial_positions['joint_a1']}</param>
-                </state_interface>
-                <state_interface name="velocity">
-                    <param name="initial_value">0.0</param>
-                </state_interface>
-                <state_interface name="effort">
-                    <param name="initial_value">0.0</param>
-                </state_interface>
-            </joint>
-            <joint name="${prefix}joint_a2">
-                <command_interface name="${command_interface}" />
-                    <xacro:if value="${command_interface == 'position'}">
-                        <param name="min">-2.09</param>
-                        <param name="max">2.09</param>
-                    </xacro:if>
-                <state_interface name="position">
-                    <param name="initial_value">${initial_positions['joint_a2']}</param>
-                </state_interface>
-                <state_interface name="velocity">
-                    <param name="initial_value">0.0</param>
-                </state_interface>
-                <state_interface name="effort">
-                    <param name="initial_value">0.0</param>
-                </state_interface>
-            </joint>
-            <joint name="${prefix}joint_a3">
-                <command_interface name="${command_interface}" />
-                    <xacro:if value="${command_interface == 'position'}">
-                        <param name="min">-2.96</param>
-                        <param name="max">2.96</param>
-                    </xacro:if>
-                <state_interface name="position">
-                    <param name="initial_value">${initial_positions['joint_a3']}</param>
-                </state_interface>
-                <state_interface name="velocity">
-                    <param name="initial_value">0.0</param>
-                </state_interface>
-                <state_interface name="effort">
-                    <param name="initial_value">0.0</param>
-                </state_interface>
-            </joint>
-            <joint name="${prefix}joint_a4">
-                <command_interface name="${command_interface}" />
-                    <xacro:if value="${command_interface == 'position'}">
-                        <param name="min">-2.09</param>
-                        <param name="max">2.09</param>
-                    </xacro:if>
-                <state_interface name="position">
-                    <param name="initial_value">${initial_positions['joint_a4']}</param>
-                </state_interface>
-                <state_interface name="velocity">
-                    <param name="initial_value">0.0</param>
-                </state_interface>
-                <state_interface name="effort">
-                    <param name="initial_value">0.0</param>
-                </state_interface>
-            </joint>
-            <joint name="${prefix}joint_a5">
-                <command_interface name="${command_interface}" />
-                    <xacro:if value="${command_interface == 'position'}">
-                        <param name="min">-2.96</param>
-                        <param name="max">2.96</param>
-                    </xacro:if>
-                <state_interface name="position">
-                    <param name="initial_value">${initial_positions['joint_a5']}</param>
-                </state_interface>
-                <state_interface name="velocity">
-                    <param name="initial_value">0.0</param>
-                </state_interface>
-                <state_interface name="effort">
-                    <param name="initial_value">0.0</param>
-                </state_interface>
-            </joint>
-            <joint name="${prefix}joint_a6">
-                <command_interface name="${command_interface}" />
-                    <xacro:if value="${command_interface == 'position'}">
-                        <param name="min">-2.09</param>
-                        <param name="max">2.09</param>
-                    </xacro:if>
-                <state_interface name="position">
-                    <param name="initial_value">${initial_positions['joint_a6']}</param>
-                </state_interface>
-                <state_interface name="velocity">
-                    <param name="initial_value">0.0</param>
-                </state_interface>
-                <state_interface name="effort">
-                    <param name="initial_value">0.0</param>
-                </state_interface>
-            </joint>
-            <joint name="${prefix}joint_a7">
-                <command_interface name="${command_interface}" />
-                    <xacro:if value="${command_interface == 'position'}">
-                        <param name="min">-3.05</param>
-                        <param name="max">3.05</param>
-                    </xacro:if>
-                <state_interface name="position">
-                    <param name="initial_value">${initial_positions['joint_a7']}</param>
-                </state_interface>
-                <state_interface name="velocity">
-                    <param name="initial_value">0.0</param>
-                </state_interface>
-                <state_interface name="effort">
-                    <param name="initial_value">0.0</param>
-                </state_interface>
-            </joint>
-            <sensor name="${prefix}external_torque_sensor">
-                <state_interface name="external_torque.joint_a1"/>
-                <state_interface name="external_torque.joint_a2"/>
-                <state_interface name="external_torque.joint_a3"/>
-                <state_interface name="external_torque.joint_a4"/>
-                <state_interface name="external_torque.joint_a5"/>
-                <state_interface name="external_torque.joint_a6"/>
-                <state_interface name="external_torque.joint_a7"/>
-            </sensor>
-        </ros2_control>
+            <state_interface name="position">
+                <param name="initial_value">0</param>
+            </state_interface>
+            <state_interface name="velocity">
+                <param name="initial_value">0.0</param>
+            </state_interface>
+            <state_interface name="effort">
+                <param name="initial_value">0.0</param>
+            </state_interface>
+        </joint>
+        <joint name="${prefix}joint_a2">
+            <command_interface name="${command_interface}" />
+            <xacro:if value="${command_interface == 'position'}">
+                <param name="min">-2.09</param>
+                <param name="max">2.09</param>
+            </xacro:if>
+            <state_interface name="position">
+                <param name="initial_value">0</param>
+            </state_interface>
+            <state_interface name="velocity">
+                <param name="initial_value">0.0</param>
+            </state_interface>
+            <state_interface name="effort">
+                <param name="initial_value">0.0</param>
+            </state_interface>
+        </joint>
+        <joint name="${prefix}joint_a3">
+            <command_interface name="${command_interface}" />
+            <xacro:if value="${command_interface == 'position'}">
+                <param name="min">-2.96</param>
+                <param name="max">2.96</param>
+            </xacro:if>
+            <state_interface name="position">
+                <param name="initial_value">0</param>
+            </state_interface>
+            <state_interface name="velocity">
+                <param name="initial_value">0.0</param>
+            </state_interface>
+            <state_interface name="effort">
+                <param name="initial_value">0.0</param>
+            </state_interface>
+        </joint>
+        <joint name="${prefix}joint_a4">
+            <command_interface name="${command_interface}" />
+            <xacro:if value="${command_interface == 'position'}">
+                <param name="min">-2.09</param>
+                <param name="max">2.09</param>
+            </xacro:if>
+            <state_interface name="position">
+                <param name="initial_value">0</param>
+            </state_interface>
+            <state_interface name="velocity">
+                <param name="initial_value">0.0</param>
+            </state_interface>
+            <state_interface name="effort">
+                <param name="initial_value">0.0</param>
+            </state_interface>
+        </joint>
+        <joint name="${prefix}joint_a5">
+            <command_interface name="${command_interface}" />
+            <xacro:if value="${command_interface == 'position'}">
+                <param name="min">-2.96</param>
+                <param name="max">2.96</param>
+            </xacro:if>
+            <state_interface name="position">
+                <param name="initial_value">0</param>
+            </state_interface>
+            <state_interface name="velocity">
+                <param name="initial_value">0.0</param>
+            </state_interface>
+            <state_interface name="effort">
+                <param name="initial_value">0.0</param>
+            </state_interface>
+        </joint>
+        <joint name="${prefix}joint_a6">
+            <command_interface name="${command_interface}" />
+            <xacro:if value="${command_interface == 'position'}">
+                <param name="min">-2.09</param>
+                <param name="max">2.09</param>
+            </xacro:if>
+            <state_interface name="position">
+                <param name="initial_value">0</param>
+            </state_interface>
+            <state_interface name="velocity">
+                <param name="initial_value">0.0</param>
+            </state_interface>
+            <state_interface name="effort">
+                <param name="initial_value">0.0</param>
+            </state_interface>
+        </joint>
+        <joint name="${prefix}joint_a7">
+            <command_interface name="${command_interface}" />
+            <xacro:if value="${command_interface == 'position'}">
+                <param name="min">-3.05</param>
+                <param name="max">3.05</param>
+            </xacro:if>
+            <state_interface name="position">
+                <param name="initial_value">0</param>
+            </state_interface>
+            <state_interface name="velocity">
+                <param name="initial_value">0.0</param>
+            </state_interface>
+            <state_interface name="effort">
+                <param name="initial_value">0.0</param>
+            </state_interface>
+        </joint>
+        <sensor name="${prefix}external_torque_sensor">
+            <state_interface name="external_torque.joint_a1" />
+            <state_interface name="external_torque.joint_a2" />
+            <state_interface name="external_torque.joint_a3" />
+            <state_interface name="external_torque.joint_a4" />
+            <state_interface name="external_torque.joint_a5" />
+            <state_interface name="external_torque.joint_a6" />
+            <state_interface name="external_torque.joint_a7" />
+        </sensor>
     </xacro:macro>
 </robot>

File: victor_description/urdf/victor.urdf.xacro (robot description, xacro)
@@ -2,8 +2,16 @@
 <robot name="victor" xmlns:xacro="http://www.ros.org/wiki/xacro">
   <xacro:arg name="robot_name" default="victor"/>
+  <xacro:arg name="left_robot_ip" default="10.10.10.12" />
+  <xacro:arg name="left_robot_port" default="30200" />
+  <xacro:arg name="right_robot_ip" default="10.10.10.11" />
+  <xacro:arg name="right_robot_port" default="30200" />
+  <xacro:arg name="command_interface" default="position" />
+  <xacro:arg name="use_fake_hardware" default="false" />
+  <xacro:arg name="controllers_file" default="iiwa_controllers.yaml" />
   <xacro:include filename="$(find victor_description)/urdf/baxter_pedestal.xacro"/>
   <xacro:include filename="$(find victor_description)/urdf/victor_torso.xacro"/>
   <xacro:include filename="$(find victor_description)/urdf/iiwa.urdf.xacro"/>
   <xacro:include filename="$(find victor_description)/urdf/materials.xacro"/>
+  <xacro:include filename="$(find victor_description)/ros2_control/victor.r2c_hardware.xacro"/>
   <xacro:baxter_pedestal robot_name="$(arg robot_name)"/>
   <xacro:victor_torso robot_name="$(arg robot_name)" parent="$(arg robot_name)_base_plate_mount"/>
@@ -28,3 +36,10 @@
   <link name="$(arg robot_name)_right_arm_world_frame_kuka">
   </link>
+  <xacro:victor_r2c_hardware
+      name="victor"
+      command_interface="$(arg command_interface)"
+      left_robot_ip="$(arg left_robot_ip)" left_robot_port="$(arg left_robot_port)"
+      right_robot_ip="$(arg right_robot_ip)" right_robot_port="$(arg right_robot_port)"
+      use_fake_hardware="$(arg use_fake_hardware)"
+      />
 </robot>
