Commit message: disable ETS because I currently think it is duplicative with the publish joint effort??

File: victor_description/srdf/iiwa_macro.srdf.xacro (robot description, xacro)
@@ -1,48 +1,48 @@
 <?xml version="1.0"?>
 <robot xmlns:xacro="http://www.ros.org/wiki/xacro">
-  <xacro:macro name="victor_srdf" params="name prefix">
-     <group name="${prefix}${name}_arm">
-        <chain base_link="${prefix}victor_base" tip_link="${prefix}tool0" />
-    </group>
-    <group_state name="ready" group="${prefix}${name}_arm">
-        <joint name="${prefix}joint_a1" value="0"/>
-        <joint name="${prefix}joint_a2" value="-0.785"/>
-        <joint name="${prefix}joint_a3" value="0"/>
-        <joint name="${prefix}joint_a4" value="-2.356"/>
-        <joint name="${prefix}joint_a5" value="0"/>
-        <joint name="${prefix}joint_a6" value="1.571"/>
-        <joint name="${prefix}joint_a7" value="0.785"/>
-    </group_state>
-    <virtual_joint child_link="${prefix}victor_base" name="virtual_joint" parent_frame="world" type="floating"/>
-    <disable_collisions link1="${prefix}victor_base" link2="${prefix}link_0" reason="Adjacent" />
-    <disable_collisions link1="${prefix}victor_base" link2="${prefix}link_1" reason="Never" />
-    <disable_collisions link1="${prefix}victor_base" link2="${prefix}link_2" reason="Never" />
-    <disable_collisions link1="${prefix}victor_base" link2="${prefix}link_3" reason="Never" />
-    <disable_collisions link1="${prefix}link_0" link2="${prefix}link_1" reason="Adjacent" />
-    <disable_collisions link1="${prefix}link_0" link2="${prefix}link_2" reason="Never" />
-    <disable_collisions link1="${prefix}link_0" link2="${prefix}link_3" reason="Never" />
-    <disable_collisions link1="${prefix}link_0" link2="${prefix}link_4" reason="Never" />
-    <disable_collisions link1="${prefix}link_1" link2="${prefix}link_2" reason="Adjacent" />
-    <disable_collisions link1="${prefix}link_1" link2="${prefix}link_3" reason="Never" />
-    <disable_collisions link1="${prefix}link_1" link2="${prefix}link_4" reason="Never" />
-    <disable_collisions link1="${prefix}link_1" link2="${prefix}link_5" reason="Never" />
-    <disable_collisions link1="${prefix}link_1" link2="${prefix}link_6" reason="Never" />
-    <disable_collisions link1="${prefix}link_1" link2="${prefix}link_7" reason="Never" />
-    <disable_collisions link1="${prefix}link_2" link2="${prefix}link_3" reason="Adjacent" />
-    <disable_collisions link1="${prefix}link_2" link2="${prefix}link_4" reason="Never" />
-    <disable_collisions link1="${prefix}link_2" link2="${prefix}link_5" reason="Never" />
-    <disable_collisions link1="${prefix}link_2" link2="${prefix}link_6" reason="Never" />
-    <disable_collisions link1="${prefix}link_2" link2="${prefix}link_7" reason="Never" />
-    <disable_collisions link1="${prefix}link_3" link2="${prefix}link_4" reason="Adjacent" />
-    <disable_collisions link1="${prefix}link_3" link2="${prefix}link_5" reason="Never" />
-    <disable_collisions link1="${prefix}link_3" link2="${prefix}link_6" reason="Never" />
-    <disable_collisions link1="${prefix}link_3" link2="${prefix}link_7" reason="Never" />
-    <disable_collisions link1="${prefix}link_4" link2="${prefix}link_5" reason="Adjacent" />
-    <disable_collisions link1="${prefix}link_4" link2="${prefix}link_6" reason="Never" />
-    <disable_collisions link1="${prefix}link_4" link2="${prefix}link_7" reason="Never" />
-    <disable_collisions link1="${prefix}link_5" link2="${prefix}link_6" reason="Adjacent" />
-    <disable_collisions link1="${prefix}link_5" link2="${prefix}link_7" reason="Never" />
-    <disable_collisions link1="${prefix}link_6" link2="${prefix}link_7" reason="Adjacent" />
-    <disable_collisions link1="${prefix}link_7" link2="${prefix}tool0" reason="Adjacent" />
-  </xacro:macro>
+    <xacro:macro name="iiwa_srdf" params="prefix">
+        <group name="${prefix}arm">
+            <chain base_link="${prefix}victor_base" tip_link="${prefix}tool0"/>
+        </group>
+        <group_state name="zero" group="${prefix}arm">
+            <joint name="${prefix}joint_a1" value="0"/>
+            <joint name="${prefix}joint_a2" value="0"/>
+            <joint name="${prefix}joint_a3" value="0"/>
+            <joint name="${prefix}joint_a4" value="0"/>
+            <joint name="${prefix}joint_a5" value="0"/>
+            <joint name="${prefix}joint_a6" value="0"/>
+            <joint name="${prefix}joint_a7" value="0"/>
+        </group_state>
+        <virtual_joint child_link="${prefix}victor_base" name="virtual_joint" parent_frame="world" type="floating"/>
+        <disable_collisions link1="${prefix}victor_base" link2="${prefix}link_0" reason="Adjacent"/>
+        <disable_collisions link1="${prefix}victor_base" link2="${prefix}link_1" reason="Never"/>
+        <disable_collisions link1="${prefix}victor_base" link2="${prefix}link_2" reason="Never"/>
+        <disable_collisions link1="${prefix}victor_base" link2="${prefix}link_3" reason="Never"/>
+        <disable_collisions link1="${prefix}link_0" link2="${prefix}link_1" reason="Adjacent"/>
+        <disable_collisions link1="${prefix}link_0" link2="${prefix}link_2" reason="Never"/>
+        <disable_collisions link1="${prefix}link_0" link2="${prefix}link_3" reason="Never"/>
+        <disable_collisions link1="${prefix}link_0" link2="${prefix}link_4" reason="Never"/>
+        <disable_collisions link1="${prefix}link_1" link2="${prefix}link_2" reason="Adjacent"/>
+        <disable_collisions link1="${prefix}link_1" link2="${prefix}link_3" reason="Never"/>
+        <disable_collisions link1="${prefix}link_1" link2="${prefix}link_4" reason="Never"/>
+        <disable_collisions link1="${prefix}link_1" link2="${prefix}link_5" reason="Never"/>
+        <disable_collisions link1="${prefix}link_1" link2="${prefix}link_6" reason="Never"/>
+        <disable_collisions link1="${prefix}link_1" link2="${prefix}link_7" reason="Never"/>
+        <disable_collisions link1="${prefix}link_2" link2="${prefix}link_3" reason="Adjacent"/>
+        <disable_collisions link1="${prefix}link_2" link2="${prefix}link_4" reason="Never"/>
+        <disable_collisions link1="${prefix}link_2" link2="${prefix}link_5" reason="Never"/>
+        <disable_collisions link1="${prefix}link_2" link2="${prefix}link_6" reason="Never"/>
+        <disable_collisions link1="${prefix}link_2" link2="${prefix}link_7" reason="Never"/>
+        <disable_collisions link1="${prefix}link_3" link2="${prefix}link_4" reason="Adjacent"/>
+        <disable_collisions link1="${prefix}link_3" link2="${prefix}link_5" reason="Never"/>
+        <disable_collisions link1="${prefix}link_3" link2="${prefix}link_6" reason="Never"/>
+        <disable_collisions link1="${prefix}link_3" link2="${prefix}link_7" reason="Never"/>
+        <disable_collisions link1="${prefix}link_4" link2="${prefix}link_5" reason="Adjacent"/>
+        <disable_collisions link1="${prefix}link_4" link2="${prefix}link_6" reason="Never"/>
+        <disable_collisions link1="${prefix}link_4" link2="${prefix}link_7" reason="Never"/>
+        <disable_collisions link1="${prefix}link_5" link2="${prefix}link_6" reason="Adjacent"/>
+        <disable_collisions link1="${prefix}link_5" link2="${prefix}link_7" reason="Never"/>
+        <disable_collisions link1="${prefix}link_6" link2="${prefix}link_7" reason="Adjacent"/>
+        <disable_collisions link1="${prefix}link_7" link2="${prefix}tool0" reason="Adjacent"/>
+    </xacro:macro>
 </robot>

Commit message: update docs and working on moveit config

File: victor_description/srdf/iiwa_macro.srdf.xacro (robot description, xacro)
@@ -14,5 +14,4 @@
             <joint name="${prefix}joint_a7" value="0"/>
         </group_state>
-        <virtual_joint child_link="${prefix}victor_base" name="virtual_joint" parent_frame="world" type="floating"/>
         <disable_collisions link1="${prefix}victor_base" link2="${prefix}link_0" reason="Adjacent"/>
         <disable_collisions link1="${prefix}victor_base" link2="${prefix}link_1" reason="Never"/>

File: victor_description/srdf/victor.srdf.xacro (robot description, xacro)
@@ -12,18 +12,18 @@
   </group>
   <group_state name="impedance_switch" group="both_arms">
-    <joint name="victor_left_arm_joint_1" value="-0.694"/>
-    <joint name="victor_left_arm_joint_2" value="0.140"/>
-    <joint name="victor_left_arm_joint_3" value="-0.229"/>
-    <joint name="victor_left_arm_joint_4" value="-1.110"/>
-    <joint name="victor_left_arm_joint_5" value="-0.512"/>
-    <joint name="victor_left_arm_joint_6" value="1.272"/>
-    <joint name="victor_left_arm_joint_7" value="0.077"/>
-    <joint name="victor_right_arm_joint_1" value="0.724"/>
-    <joint name="victor_right_arm_joint_2" value="0.451"/>
-    <joint name="victor_right_arm_joint_3" value="0.940"/>
-    <joint name="victor_right_arm_joint_4" value="-1.425"/>
-    <joint name="victor_right_arm_joint_5" value="0.472"/>
-    <joint name="victor_right_arm_joint_6" value="0.777"/>
-    <joint name="victor_right_arm_joint_7" value="-0.809"/>
+    <joint name="left_joint_a1" value="-0.694"/>
+    <joint name="left_joint_a2" value="0.140"/>
+    <joint name="left_joint_a3" value="-0.229"/>
+    <joint name="left_joint_a4" value="-1.110"/>
+    <joint name="left_joint_a5" value="-0.512"/>
+    <joint name="left_joint_a6" value="1.272"/>
+    <joint name="left_joint_a7" value="0.077"/>
+    <joint name="right_joint_a1" value="0.724"/>
+    <joint name="right_joint_a2" value="0.451"/>
+    <joint name="right_joint_a3" value="0.940"/>
+    <joint name="right_joint_a4" value="-1.425"/>
+    <joint name="right_joint_a5" value="0.472"/>
+    <joint name="right_joint_a6" value="0.777"/>
+    <joint name="right_joint_a7" value="-0.809"/>
   </group_state>
 </robot>
